File: urban battery - power_distribution.kicad_sch (KiCad schematic)
At the start: 23 parts, among them J1 FRONT_ACC_OUT, J2 12V_IN, J3 12VHC_OUT_EXTRA, J4 TEL_OUT, J5 REAR_ACC_OUT, J6 MTR_CTRL_OUT, J7 12VLC_OUT_EXTRA, J8 12VLC_OUT_EXTRA, J9 12VLC_OUT_EXTRA

Commit message: fixed schematic and layout bugs
Parts:
- removed H3, H4: MountingHole, MountingHole:MountingHole_3.2mm_M3, symbol Mechanical:MountingHole
Changed lines of the file:
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@@
-    )
-  )
-  (symbol (lib_id "Mechanical:MountingHole") (at 116.84 177.165 0) (unit 1)
-    (in_bom yes) (on_board yes) (fields_autoplaced)
-    (property "Reference" "H3" (id 0) (at 119.38 175.8949 0)
-      (effects (font (size 1.27 1.27)) (justify left))
-    )
-    (property "Value" "MountingHole" (id 1) (at 119.38 178.4349 0)
-      (effects (font (size 1.27 1.27)) (justify left))
-    )
-    (property "Footprint" "MountingHole:MountingHole_3.2mm_M3" (id 2) (at 116.84 177.165 0)
-      (effects (font (size 1.27 1.27)) hide)
-    )
-    (property "Datasheet" "~" (id 3) (at 116.84 177.165 0)
-      (effects (font (size 1.27 1.27)) hide)
     )
   )
@@
     (pin "2")
   )
-  (symbol (lib_id "Mechanical:MountingHole") (at 116.84 184.15 0) (unit 1)
-    (in_bom yes) (on_board yes) (fields_autoplaced)
-    (property "Reference" "H4" (id 0) (at 119.38 182.8799 0)
-      (effects (font (size 1.27 1.27)) (justify left))
-    )
-    (property "Value" "MountingHole" (id 1) (at 119.38 185.4199 0)
-      (effects (font (size 1.27 1.27)) (justify left))
-    )
-    (property "Footprint" "MountingHole:MountingHole_3.2mm_M3" (id 2) (at 116.84 184.15 0)
-      (effects (font (size 1.27 1.27)) hide)
-    )
-    (property "Datasheet" "~" (id 3) (at 116.84 184.15 0)
-      (effects (font (size 1.27 1.27)) hide)
-    )
-  )
   (symbol (lib_id "Device:Fuse") (at 207.645 100.965 90) (unit 1)
     (in_bom yes) (on_board yes) (fields_autoplaced)
@@
       (reference "H2") (unit 1) (value "MountingHole") (footprint "MountingHole:MountingHole_3.2mm_M3")
     )
-    (path "/978647d5-c0bc-48a8-9c14-521d2789a3c2"
-      (reference "H3") (unit 1) (value "MountingHole") (footprint "MountingHole:MountingHole_3.2mm_M3")
-    )
-    (path "/de2f7f65-a407-4d54-bc38-1d880d70997b"
-      (reference "H4") (unit 1) (value "MountingHole") (footprint "MountingHole:MountingHole_3.2mm_M3")
-    )
     (path "/ffaacf94-8060-464b-8e0a-8714b7727bc4"
