File: urban battery - power_distribution.kicad_pcb (KiCad board)
At the start: 2 copper layers, 88.3 x 71.1 mm, 22 parts, among them J1 FRONT_ACC_OUT, J2 12V_IN, J3 12VHC_OUT_EXTRA, J4 TEL_OUT, J5 REAR_ACC_OUT, J6 MTR_CTRL_OUT, J7 12VLC_OUT_EXTRA, J8 12VLC_OUT_EXTRA, J9 12VLC_OUT_EXTRA

Commit message: final layout touches
Parts:
- J5: value REAR_ACC_OUT -> REAR ACC
- moved F5 1.27 mm to (97.7, 123.6)
- moved F4 0.84 mm to (134.6, 120.9)
- moved F1 0.63 mm to (119.6, 109.8)
- moved G*** 0.63 mm to (116.2, 125.7)
- moved J6 0.63 mm to (82.1, 124.1)
Routing:
- net Net-(F4-Pad2): track 10.8 -> 11.5 mm
- net Net-(F1-Pad2): track 31.7 -> 31.1 mm
Changed lines of the file:
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@@
   )
   (footprint "Connector_Molex:Molex_Micro-Fit_3.0_43650-0200_1x02_P3.00mm_Horizontal" (layer "F.Cu")
-    (at 82.075 124.69 90)
+    (at 82.075 124.055 90)
     (descr "Molex Micro-Fit 3.0 Connector System, 43650-0200 (compatible alternatives: 43650-0201, 43650-0202), 2 Pins per row (https://www.molex.com/pdm_docs/sd/436500300_sd.pdf), generated with kicad-footprint-generator")
     (tags "connector Molex Micro-Fit_3.0 top entry")
@@
   )
   (footprint "LOGO" (layer "F.Cu")
-    (at 116.205 126.365)
+    (at 116.205 125.73)
     (attr board_only exclude_from_pos_files exclude_from_bom)
     (fp_text reference "G***" (at 0 -1.27) (layer "F.Fab")
@@
   )
   (footprint "Fuse:Fuseholder_Blade_Mini_Keystone_3568" (layer "F.Cu")
-    (at 119.629184 109.126 75)
+    (at 119.629184 109.761 75)
     (descr "fuse holder, car blade fuse mini, http://www.keyelco.com/product-pdf.cfm?p=306")
     (tags "car blade fuse mini")
@@
   )
   (footprint "Fuse:Fuseholder_Blade_Mini_Keystone_3568" (layer "F.Cu")
-    (at 97.67 124.89 180)
+    (at 97.67 123.62 180)
     (descr "fuse holder, car blade fuse mini, http://www.keyelco.com/product-pdf.cfm?p=306")
     (tags "car blade fuse mini")
@@
       (effects (font (size 1 1) (thickness 0.15)))
     )
-    (fp_text value "REAR_ACC_OUT" (at 1.705 19.525 90) (layer "F.SilkS")
+    (fp_text value "REAR ACC" (at 0.865 19.525 90) (layer "F.SilkS")
       (effects (font (size 0.7 0.7) (thickness 0.15)))
     )
@@
   )
   (footprint "Fuse:Fuseholder_Blade_Mini_Keystone_3568" (layer "F.Cu")
-    (at 134.62 121.695)
+    (at 134.62 120.855)
     (descr "fuse holder, car blade fuse mini, http://www.keyelco.com/product-pdf.cfm?p=306")
     (tags "car blade fuse mini")
@@
       (effects (font (size 1 1) (thickness 0.15)))
     )
-    (fp_text value "487K" (at -2.54 0 180) (layer "F.Fab")
+    (fp_text value "487K" (at 2.7375 0 180) (layer "F.Fab")
       (effects (font (size 0.5 0.5) (thickness 0.125)))
     )
@@
   (gr_line (start 118.11 104.775) (end 113.665 104.775) (layer "Edge.Cuts") (width 0.1))
   (gr_line (start 139.065 127.548376) (end 160.02 128.905) (layer "Edge.Cuts") (width 0.1))
-  (gr_arc (start 95.25 127) (mid 95.446196 127.3175) (end 95.25 127.635) (layer "Edge.Cuts") (width 0.1))
+  (gr_arc (start 95.25 127) (mid 95.446197 127.3175) (end 95.25 127.635) (layer "Edge.Cuts") (width 0.1))
   (gr_line (start 95.25 127.635) (end 74.93 146.05) (layer "Edge.Cuts") (width 0.1))
   (gr_line (start 94.615 92.71) (end 83.185 99.06) (layer "Edge.Cuts") (width 0.1))
@@
     (effects (font (size 0.7 0.7) (thickness 0.15)))
   )
-  (gr_text "Sarah Qadar\nPower Distribution V1.0\nShell Eco-Marathon 2023" (at 116.84 114.935) (layer "F.SilkS")
+  (gr_text "Sarah Qadar\nPower Distribution V1.0\nShell Eco-Marathon 2023" (at 116.205 114.3) (layer "F.SilkS")
     (effects (font (size 0.5 0.5) (thickness 0.1)))
   )
-  (gr_text "MOTOR CNTRL" (at 101.6 123.19 270) (layer "F.SilkS")
+  (gr_text "MOTOR CNTRL" (at 101.6 121.92 270) (layer "F.SilkS")
     (effects (font (size 0.7 0.7) (thickness 0.15)))
   )
@@
   (segment (start 119.629184 109.126) (end 122.033347 109.126) (width 6.78) (layer "F.Cu") (net 1))
   (segment (start 122.033347 109.126) (end 122.913332 110.005985) (width 6.78) (layer "F.Cu") (net 1))
-  (segment (start 131.022497 109.695466) (end 131.022497 105.965681) (width 3.4) (layer "F.Cu") (net 2))
-  (segment (start 131.022497 105.965681) (end 125.480817 100.424001) (width 3.4) (layer "F.Cu") (net 2))
-  (segment (start 122.196669 99.544016) (end 124.600832 99.544016) (width 3.4) (layer "F.Cu") (net 2))
-  (segment (start 124.600832 99.544016) (end 125.480817 100.424001) (width 3.4) (layer "F.Cu") (net 2))
+  (segment (start 131.022497 105.965681) (end 131.022497 109.695466) (width 3.4) (layer "F.Cu") (net 2))
+  (segment (start 125.235832 100.179016) (end 131.022497 105.965681) (width 3.4) (layer "F.Cu") (net 2))
+  (segment (start 122.196669 100.179016) (end 125.235832 100.179016) (width 3.4) (layer "F.Cu") (net 2))
   (segment (start 122.441654 99.789001) (end 121.561669 98.909016) (width 0.5) (layer "F.Cu") (net 2))
-  (segment (start 122.347653 99.695) (end 122.196669 99.544016) (width 3.4) (layer "B.Cu") (net 2))
-  (segment (start 125.480817 100.424001) (end 124.751816 99.695) (width 3.4) (layer "B.Cu") (net 2))
+  (segment (start 125.235832 100.179016) (end 122.196669 100.179016) (width 3.4) (layer "B.Cu") (net 2))
   (segment (start 131.022497 109.695466) (end 131.022497 105.965681) (width 3.4) (layer "B.Cu") (net 2))
-  (segment (start 124.751816 99.695) (end 122.347653 99.695) (width 3.4) (layer "B.Cu") (net 2))
-  (segment (start 131.022497 105.965681) (end 125.480817 100.424001) (width 3.4) (layer "B.Cu") (net 2))
+  (segment (start 131.022497 105.965681) (end 125.235832 100.179016) (width 3.4) (layer "B.Cu") (net 2))
   (segment (start 96.364534 113.185466) (end 96.52 113.03) (width 0.5) (layer "F.Cu") (net 3))
   (segment (start 96.52 110.640261) (end 106.981246 100.179015) (width 3.85) (layer "F.Cu") (net 3))
@@
   (segment (start 148.748446 141.547126) (end 147.165651 139.964331) (width 2.89) (layer "F.Cu") (net 4))
   (segment (start 148.748446 141.547126) (end 148.055572 142.24) (width 0.25) (layer "F.Cu") (net 4))
-  (segment (start 150.33 121.695) (end 147.94 121.695) (width 2.89) (layer "F.Cu") (net 5))
-  (segment (start 144.78 125.095) (end 144.54 125.095) (width 0.25) (layer "F.Cu") (net 5))
-  (segment (start 144.54 125.095) (end 144.54 121.695) (width 2.89) (layer "F.Cu") (net 5))
+  (segment (start 144.78 125.095) (end 144.78 124.7) (width 0.25) (layer "F.Cu") (net 5))
+  (segment (start 144.54 124.065) (end 146.91 121.695) (width 2.89) (layer "F.Cu") (net 5))
   (segment (start 150.335 121.69) (end 150.33 121.695) (width 0.25) (layer "F.Cu") (net 5))
-  (segment (start 147.94 121.695) (end 144.54 125.095) (width 2.89) (layer "F.Cu") (net 5))
-  (segment (start 87.75 121.49) (end 87.75 124.89) (width 2.89) (layer "F.Cu") (net 6))
-  (segment (start 84.55 124.69) (end 87.75 121.49) (width 2.89) (layer "F.Cu") (net 6))
-  (segment (start 82.075 124.69) (end 84.55 124.69) (width 2.89) (layer "F.Cu") (net 6))
+  (segment (start 146.91 121.695) (end 150.33 121.695) (width 2.89) (layer "F.Cu") (net 5))
+  (segment (start 144.54 124.46) (end 144.54 120.855) (width 2.89) (layer "F.Cu") (net 5))
+  (segment (start 144.78 124.7) (end 144.54 124.46) (width 0.25) (layer "F.Cu") (net 5))
+  (segment (start 144.54 124.46) (end 144.54 124.065) (width 2.89) (layer "F.Cu") (net 5))
+  (segment (start 82.075 124.055) (end 83.915 124.055) (width 2.89) (layer "F.Cu") (net 6))
+  (segment (start 87.75 120.22) (end 87.75 123.62) (width 2.89) (layer "F.Cu") (net 6))
+  (segment (start 83.915 124.055) (end 87.75 120.22) (width 2.89) (layer "F.Cu") (net 6))
   (segment (start 87.687874 143.668446) (end 89.27067 142.08565) (width 2.89) (layer "F.Cu") (net 7))
   (segment (start 89.27067 142.08565) (end 89.27067 137.560168) (width 2.89) (layer "F.Cu") (net 7))
