File: urban battery - power_distribution.kicad_pcb (KiCad board)
At the start: 2 copper layers, 88.3 x 71.1 mm, 22 parts, among them J1 FRONT_ACC_OUT, J2 12V_IN, J3 12VHC_OUT_EXTRA, J4 TEL_OUT, J5 REAR ACC, J6 MTR_CTRL_OUT, J7 12VLC_OUT_EXTRA, J8 12VLC_OUT_EXTRA, J9 12VLC_OUT_EXTRA

Commit message: generated gerbers and drill file
Parts:
- moved G*** 0.90 mm to (116.8, 125.1)
Other:
- board text added: "Sarah Qadar Shell Eco-Marathon 2023"
- board text added: "Spidey V1.0"
- board text removed: "Sarah Qadar Power Distribution V1.0 Shell Eco-Marathon 2023"
Changed lines of the file:
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@@
       (layerselection 0x00010fc_ffffffff)
       (disableapertmacros false)
-      (usegerberextensions false)
-      (usegerberattributes true)
-      (usegerberadvancedattributes true)
-      (creategerberjobfile true)
+      (usegerberextensions true)
+      (usegerberattributes false)
+      (usegerberadvancedattributes false)
+      (creategerberjobfile false)
       (svguseinch false)
       (svgprecision 6)
@@
       (plotinvisibletext false)
       (sketchpadsonfab false)
-      (subtractmaskfromsilk false)
+      (subtractmaskfromsilk true)
       (outputformat 1)
       (mirror false)
-      (drillshape 1)
+      (drillshape 0)
       (scaleselection 1)
-      (outputdirectory "")
+      (outputdirectory "gerbers/")
     )
   )
@@
     (fp_line (start 0 0) (end 0.75 0.98) (layer "F.Fab") (width 0.1))
     (pad "" np_thru_hole circle (at 1.5 -4.32 150) (size 3 3) (drill 3) (layers *.Cu *.Mask))
-    (pad "1" thru_hole roundrect (at 0 0 150) (size 1.5 2.02) (drill 1.02) (layers *.Cu *.Mask) (roundrect_rratio 0.166667)
+    (pad "1" thru_hole roundrect (at 0 0 150) (size 1.5 2.02) (drill 1.02) (layers *.Cu *.Mask) (roundrect_rratio 0.1666673333)
       (net 8 "Net-(F7-Pad2)") (pinfunction "Pin_1") (pintype "passive"))
     (pad "2" thru_hole oval (at 3 0 150) (size 1.5 2.02) (drill 1.02) (layers *.Cu *.Mask)
@@
     (fp_line (start 5.325 -8.92) (end 6.325 -7.92) (layer "F.Fab") (width 0.1))
     (pad "" np_thru_hole circle (at 1.5 -4.32 90) (size 3 3) (drill 3) (layers *.Cu *.Mask))
-    (pad "1" thru_hole roundrect (at 0 0 90) (size 1.5 2.02) (drill 1.02) (layers *.Cu *.Mask) (roundrect_rratio 0.166667)
+    (pad "1" thru_hole roundrect (at 0 0 90) (size 1.5 2.02) (drill 1.02) (layers *.Cu *.Mask) (roundrect_rratio 0.1666673333)
       (net 6 "Net-(F5-Pad2)") (pinfunction "Pin_1") (pintype "passive"))
     (pad "2" thru_hole oval (at 3 0 90) (size 1.5 2.02) (drill 1.02) (layers *.Cu *.Mask)
@@
   )
   (footprint "LOGO" (layer "F.Cu")
-    (at 116.205 125.73)
+    (at 116.84 125.095)
     (attr board_only exclude_from_pos_files exclude_from_bom)
     (fp_text reference "G***" (at 0 -1.27) (layer "F.Fab")
@@
     (fp_line (start 5.325 -8.92) (end 6.325 -7.92) (layer "F.Fab") (width 0.1))
     (pad "" np_thru_hole circle (at 1.5 -4.32 135) (size 3 3) (drill 3) (layers *.Cu *.Mask))
-    (pad "1" thru_hole roundrect (at 0 0 135) (size 1.5 2.02) (drill 1.02) (layers *.Cu *.Mask) (roundrect_rratio 0.166667)
+    (pad "1" thru_hole roundrect (at 0 0 135) (size 1.5 2.02) (drill 1.02) (layers *.Cu *.Mask) (roundrect_rratio 0.1666673333)
       (net 7 "Net-(F6-Pad2)") (pinfunction "Pin_1") (pintype "passive"))
     (pad "2" thru_hole oval (at 3 0 135) (size 1.5 2.02) (drill 1.02) (layers *.Cu *.Mask)
@@
     (fp_line (start -2.325 -8.92) (end 5.325 -8.92) (layer "F.Fab") (width 0.1))
     (pad "" np_thru_hole circle (at 1.5 -4.32 270) (size 3 3) (drill 3) (layers *.Cu *.Mask))
-    (pad "1" thru_hole roundrect (at 0 0 270) (size 1.5 2.02) (drill 1.02) (layers *.Cu *.Mask) (roundrect_rratio 0.166667)
+    (pad "1" thru_hole roundrect (at 0 0 270) (size 1.5 2.02) (drill 1.02) (layers *.Cu *.Mask) (roundrect_rratio 0.1666673333)
       (net 5 "Net-(F4-Pad2)") (pinfunction "Pin_1") (pintype "passive"))
     (pad "2" thru_hole oval (at 3 0 270) (size 1.5 2.02) (drill 1.02) (layers *.Cu *.Mask)
@@
     (fp_line (start 6.325 -7.92) (end 6.325 0.98) (layer "F.Fab") (width 0.1))
     (pad "" np_thru_hole circle (at 1.5 -4.32 210) (size 3 3) (drill 3) (layers *.Cu *.Mask))
-    (pad "1" thru_hole roundrect (at 0 0 210) (size 1.5 2.02) (drill 1.02) (layers *.Cu *.Mask) (roundrect_rratio 0.166667)
+    (pad "1" thru_hole roundrect (at 0 0 210) (size 1.5 2.02) (drill 1.02) (layers *.Cu *.Mask) (roundrect_rratio 0.1666673333)
       (net 9 "Net-(F8-Pad2)") (pinfunction "Pin_1") (pintype "passive"))
     (pad "2" thru_hole oval (at 3 0 210) (size 1.5 2.02) (drill 1.02) (layers *.Cu *.Mask)
@@
     (fp_line (start -3.325 -7.92) (end -2.325 -8.92) (layer "F.Fab") (width 0.1))
     (pad "" np_thru_hole circle (at 1.5 -4.32 225) (size 3 3) (drill 3) (layers *.Cu *.Mask))
-    (pad "1" thru_hole roundrect (at 0 0 225) (size 1.5 2.02) (drill 1.02) (layers *.Cu *.Mask) (roundrect_rratio 0.166667)
+    (pad "1" thru_hole roundrect (at 0 0 225) (size 1.5 2.02) (drill 1.02) (layers *.Cu *.Mask) (roundrect_rratio 0.1666673333)
       (net 4 "Net-(F3-Pad2)") (pinfunction "Pin_1") (pintype "passive"))
     (pad "2" thru_hole oval (at 3 0 225) (size 1.5 2.02) (drill 1.02) (layers *.Cu *.Mask)
@@
     (fp_line (start 1 -0.625) (end 1 0.625) (layer "F.Fab") (width 0.1))
     (fp_line (start 1 0.625) (end -1 0.625) (layer "F.Fab") (width 0.1))
-    (pad "1" smd roundrect (at -0.9125 0 90) (size 1.025 1.4) (layers "F.Cu" "F.Paste" "F.Mask") (roundrect_rratio 0.243902)
+    (pad "1" smd roundrect (at -0.9125 0 90) (size 1.025 1.4) (layers "F.Cu" "F.Paste" "F.Mask") (roundrect_rratio 0.243902439)
       (net 11 "Net-(D1-Pad2)") (pintype "passive"))
-    (pad "2" smd roundrect (at 0.9125 0 90) (size 1.025 1.4) (layers "F.Cu" "F.Paste" "F.Mask") (roundrect_rratio 0.243902)
+    (pad "2" smd roundrect (at 0.9125 0 90) (size 1.025 1.4) (layers "F.Cu" "F.Paste" "F.Mask") (roundrect_rratio 0.243902439)
       (net 1 "+12V") (pintype "passive"))
     (model "${KICAD6_3DMODEL_DIR}/Resistor_SMD.3dshapes/R_0805_2012Metric.wrl"
@@
     (effects (font (size 0.7 0.7) (thickness 0.15)))
   )
-  (gr_text "Sarah Qadar\nPower Distribution V1.0\nShell Eco-Marathon 2023" (at 116.205 114.3) (layer "F.SilkS")
+  (gr_text "Spidey V1.0" (at 115.57 117.475) (layer "F.SilkS")
+    (effects (font (size 1.5 1.5) (thickness 0.3)))
+  )
+  (gr_text "Sarah Qadar\nShell Eco-Marathon 2023" (at 116.205 114.935) (layer "F.SilkS")
     (effects (font (size 0.5 0.5) (thickness 0.1)))
   )

Commit message: fixed clearance issue addressed by DRC
Connections:
- F2 pad 2: Net-(F2-Pad2) -> GND
- J3 pad 1: Net-(F2-Pad2) -> GND
Routing:
- net GND: track 12.8 -> 77.7 mm
- net Net-(F2-Pad2): track 42.4 -> 0.00 mm

Commit message: created gerbers
Parts:
- moved G*** 0.90 mm to (116.2, 125.7)
